File: Magisterka/WeWyAn.brd (EAGLE design)
At the start: 117.8 x 80 mm, 87 parts, among them IC1 LM324N, IC3 7805TV, IC4 LM324N, IC5 LM1117T-3.3-V, X10 22-23-2041, X11 22-23-2041, X19 22-23-2041, X20 22-23-2041, X21 22-23-2041, X28 22-23-2021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

Commit message: Pinswap in PWM CRIMP and moved several components
Parts:
- added X31: 22-23-2031, con-molex:22-23-2031
- R13, R14, R17, R20: value (none) -> 10k
- R16, R19, R22, R4: value (none) -> 20k
- X18: value (none) -> 22-23-2031; device con-molex:22-23-2061 -> con-molex:22-23-2031
- moved IC5 315.4 mm to (36.8, 72.4), turned to 90 degrees
- moved C9 267.3 mm to (83.8, 61.0)
- moved X18 247.9 mm to (-41.9, -166.4)
- moved C13 239.9 mm to (71.1, 15.2)
- moved C14 239.9 mm to (71.1, 10.2)
- moved C11 239.0 mm to (71.1, 24.1)
- moved C12 239.0 mm to (71.1, 19.1)
- moved C10 238.1 mm to (71.1, 27.9)
- moved C1 236.4 mm to (19.1, 77.5)
- moved C8 232.3 mm to (15.2, 71.1)
- moved IC3 218.3 mm to (21.6, 72.4), turned to 90 degrees
- moved C5 191.6 mm to (91.4, 26.7), turned to 90 degrees
- moved C4 185.1 mm to (91.4, 31.8), turned to 270 degrees
- moved R1 181.3 mm to (106.7, 55.9)
- moved R21 180.6 mm to (106.7, 31.8), turned to 90 degrees
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Connections:
- net DSTMIN0: now also X18.3; no longer X18.6
- net DSTMIN1: now also X18.2; no longer X18.5
- net DSTMIN2: now also X18.1; no longer X18.4
- net DSTMIN3: now also X31.3; no longer X18.3
- net DSTMIN4: now also X31.2; no longer X18.2
- net DSTMIN5: now also X31.1; no longer X18.1
- net PWM0: now also X11.1; no longer X11.2
- net PWM1: now also X11.2; no longer X11.1
- net PWM2: now also X11.3; no longer X11.4
- net PWM3: now also X11.4; no longer X11.3

Commit message: first final
Parts:
- moved X31 248.9 mm to (109.2, 39.4), turned to 180 degrees
- moved X29 245.6 mm to (11.4, 59.7)
- moved X18 239.2 mm to (80.0, 39.4), turned to 180 degrees
- moved X30 237.8 mm to (17.8, 59.7)
- moved X28 234.3 mm to (5.08, 59.7)
- moved X26 217.9 mm to (47.0, 72.4)
- moved X27 209.2 mm to (57.1, 72.4)
- moved X24 189.6 mm to (26.7, 72.4)
- moved X25 181.2 mm to (36.8, 72.4)
- moved X15 178.5 mm to (100.3, 72.4)
- moved X21 173.2 mm to (54.6, 59.7)
- moved X22 161.3 mm to (6.35, 72.4)
- moved X7 159.9 mm to (81.3, 3.81), turned to 180 degrees
- moved X14 157.2 mm to (90.2, 72.4)
- moved X20 154.0 mm to (41.9, 59.7)
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Connections:
- net DIN0+: now also R1.1; no longer OK2.1
- net DIN0-: now also OK2.1; no longer R1.1
- net DIN1+: now also R3.1; no longer OK1.1
- net DIN1-: now also OK1.1; no longer R3.1
- net DIN2+: now also R2.1; no longer OK4.1
- net DIN2-: now also OK4.1; no longer R2.1
- net DIN3+: now also R24.1; no longer OK3.1
- net DIN3-: now also OK3.1; no longer R24.1
- net DIN4+: now also R29.1; no longer OK6.1
- net DIN4-: now also OK6.1; no longer R29.1
- net DIN5+: now also R30.1; no longer OK5.1
- net DIN5-: now also OK5.1; no longer R30.1
- net DSTMIN0: now also OK2.4, R25.1; no longer R25.2
- net DSTMIN1: now also OK1.4
- net DSTMIN2: now also OK4.4, R27.1; no longer R27.2
- net DSTMIN3: now also OK3.4, R28.1; no longer R28.2
- net DSTMIN4: now also OK6.4, R31.1; no longer R31.2
- net DSTMIN5: now also OK5.4, R32.1; no longer R32.2
- net VCC: now also R25.2, R27.2, R28.2, R31.2, R32.2; no longer OK1.4, OK2.4, OK3.4, OK4.4, OK5.4, OK6.4, R25.1, R27.1, R28.1, R31.1, R32.1
Other:
- board size 117.8 x 80 mm -> 127.9 x 76.2 mm
- board text added: "H"
- board text added: "M"

Commit message: size changes
Parts:
- moved X4 23.4 mm to (97.8, 27.9), turned to 90 degrees
- moved X11 3.81 mm to (82.5, 25.4)
- moved X10 1.27 mm to (3.81, 25.4)
- moved R15 1.17 mm to (52.5, 28.7), turned to 0 degrees
- moved R23 1.17 mm to (52.6, 22.0), turned to 0 degrees
- moved R18 1.09 mm to (72.0, 22.2), turned to 180 degrees
- moved R21 0.99 mm to (71.9, 28.6), turned to 180 degrees
Routing:
- net VCC: track 0.00 -> 165.1 mm
- net VDD: track 0.00 -> 80.5 mm
- net 5V: track 0.00 -> 59.4 mm
- net PWM0: track 0.00 -> 58.8 mm
- net PWM1: track 0.00 -> 44.7 mm
- net ADC2: track 0.00 -> 43.5 mm, vias 0 -> 1
- net AOUT3: track 0.00 -> 43.0 mm
- net ADC3: track 0.00 -> 39.2 mm, vias 0 -> 1
- net AIN3: track 0.00 -> 37.1 mm
- net AOUT0: track 0.00 -> 34.8 mm
- net AIN2: track 0.00 -> 32.4 mm
- net AIN0: track 0.00 -> 30.6 mm
- net DOUT0+: track 0.00 -> 26.8 mm
- net DOUT0-: track 0.00 -> 24.3 mm
- net AIN1: track 0.00 -> 23.7 mm
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- added copper zone on layer 1, net GND
- added copper zone on layer 16, net GND
Other:
- board text added: "0"
- board text added: "ADC"
- board text added: "ANALOG IN"
- board text added: "ANALOG OUT"
- board text added: "DSTMIN"
- board text added: "GND"
- board text added: "RELAY CONN"
- board text added: "RELAY POWER"
- board text added: "VCC"

Commit message: Added relays
Parts:
- added K1, K2, K3, K4, K5, K6: E3206S, relay:E3206S
Other:
- board size 127.9 x 76.2 mm -> 175 x 108 mm
Changed lines of the file:
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@@
 <setting verticaltext="up"/>
 </settings>
-<grid distance="50" unitdist="mil" unit="mil" style="lines" multiple="1" display="no" altdistance="5" altunitdist="mil" altunit="mil"/>
+<grid distance="50" unitdist="mil" unit="mm" style="lines" multiple="1" display="no" altdistance="5" altunitdist="mil" altunit="mm"/>
 <layers>
 <layer number="1" name="Top" color="4" fill="1" visible="yes" active="yes"/>
@@
 <board>
 <plain>
-<wire x1="0" y1="0" x2="127.94" y2="0" width="0" layer="20"/>
-<wire x1="127.94" y1="0" x2="127.94" y2="76.19" width="0" layer="20"/>
-<wire x1="127.94" y1="76.19" x2="0" y2="76.19" width="0" layer="20"/>
-<wire x1="0" y1="76.19" x2="0" y2="0" width="0" layer="20"/>
+<wire x1="0" y1="0" x2="175" y2="0" width="0" layer="20"/>
+<wire x1="175" y1="0" x2="175" y2="108" width="0" layer="20"/>
+<wire x1="175" y1="108" x2="0" y2="108" width="0" layer="20"/>
+<wire x1="0" y1="108" x2="0" y2="0" width="0" layer="20"/>
 <wire x1="119.38" y1="10.16" x2="123.19" y2="10.16" width="0.1524" layer="25"/>
 <wire x1="118.745" y1="6.477" x2="120.65" y2="4.191" width="0.1524" layer="25"/>
@@
 <attribute name="OC_NEWARK" value="30C0862" x="109.22" y="39.37" size="1.778" layer="27" rot="R180" display="off"/>
 </element>
+<element name="K1" library="relay" library_urn="urn:adsk.eagle:library:339" package="E3206S" package3d_urn="urn:adsk.eagle:package:24311/1" value="E3206S" x="160.02" y="67.31">
+<attribute name="MF" value="" x="160.02" y="67.31" size="1.27" layer="27" display="off"/>
+<attribute name="MPN" value="" x="160.02" y="67.31" size="1.27" layer="27" display="off"/>
+<attribute name="OC_FARNELL" value="unknown" x="160.02" y="67.31" size="1.27" layer="27" display="off"/>
+<attribute name="OC_NEWARK" value="unknown" x="160.02" y="67.31" size="1.27" layer="27" display="off"/>
+</element>
+<element name="K2" library="relay" library_urn="urn:adsk.eagle:library:339" package="E3206S" package3d_urn="urn:adsk.eagle:package:24311/1" value="E3206S" x="149.86" y="40.64">
+<attribute name="MF" value="" x="149.86" y="40.64" size="1.27" layer="27" display="off"/>
+<attribute name="MPN" value="" x="149.86" y="40.64" size="1.27" layer="27" display="off"/>
+<attribute name="OC_FARNELL" value="unknown" x="149.86" y="40.64" size="1.27" layer="27" display="off"/>
+<attribute name="OC_NEWARK" value="unknown" x="149.86" y="40.64" size="1.27" layer="27" display="off"/>
+</element>
+<element name="K3" library="relay" library_urn="urn:adsk.eagle:library:339" package="E3206S" package3d_urn="urn:adsk.eagle:package:24311/1" value="E3206S" x="146.05" y="24.13">
+<attribute name="MF" value="" x="146.05" y="24.13" size="1.27" layer="27" display="off"/>
+<attribute name="MPN" value="" x="146.05" y="24.13" size="1.27" layer="27" display="off"/>
+<attribute name="OC_FARNELL" value="unknown" x="146.05" y="24.13" size="1.27" layer="27" display="off"/>
+<attribute name="OC_NEWARK" value="unknown" x="146.05" y="24.13" size="1.27" layer="27" display="off"/>
+</element>
+<element name="K4" library="relay" library_urn="urn:adsk.eagle:library:339" package="E3206S" package3d_urn="urn:adsk.eagle:package:24311/1" value="E3206S" x="147.32" y="8.89">
+<attribute name="MF" value="" x="147.32" y="8.89" size="1.27" layer="27" display="off"/>
+<attribute name="MPN" value="" x="147.32" y="8.89" size="1.27" layer="27" display="off"/>
+<attribute name="OC_FARNELL" value="unknown" x="147.32" y="8.89" size="1.27" layer="27" display="off"/>
+<attribute name="OC_NEWARK" value="unknown" x="147.32" y="8.89" size="1.27" layer="27" display="off"/>
+</element>
+<element name="K5" library="relay" library_urn="urn:adsk.eagle:library:339" package="E3206S" package3d_urn="urn:adsk.eagle:package:24311/1" value="E3206S" x="151.13" y="85.09">
+<attribute name="MF" value="" x="151.13" y="85.09" size="1.27" layer="27" display="off"/>
+<attribute name="MPN" value="" x="151.13" y="85.09" size="1.27" layer="27" display="off"/>
+<attribute name="OC_FARNELL" value="unknown" x="151.13" y="85.09" size="1.27" layer="27" display="off"/>
+<attribute name="OC_NEWARK" value="unknown" x="151.13" y="85.09" size="1.27" layer="27" display="off"/>
+</element>
+<element name="K6" library="relay" library_urn="urn:adsk.eagle:library:339" package="E3206S" package3d_urn="urn:adsk.eagle:package:24311/1" value="E3206S" x="153.67" y="60.96">
+<attribute name="MF" value="" x="153.67" y="60.96" size="1.27" layer="27" display="off"/>
+<attribute name="MPN" value="" x="153.67" y="60.96" size="1.27" layer="27" display="off"/>
+<attribute name="OC_FARNELL" value="unknown" x="153.67" y="60.96" size="1.27" layer="27" display="off"/>
+<attribute name="OC_NEWARK" value="unknown" x="153.67" y="60.96" size="1.27" layer="27" display="off"/>
+</element>
 </elements>

Commit message: second final
Parts:
- removed X21: 22-23-2041, con-molex:22-23-2041
- removed X28, X29, X30: 22-23-2021, con-molex:22-23-2021
- added D1, D2, D3, D4, D5, D6: (no value), diode:DO214AC
- added H1, H2, H3, H4: MOUNT-HOLE3.0, holes:3,0
- added R40, R41, R42, R43, R44, R45: (no value), rcl:R0603
- added T1, T2, T3, T4, T5, T6: (no value), zetex:SOT223
- X19, X20: value 22-23-2041 -> 22-23-2031; device con-molex:22-23-2041 -> con-molex:22-23-2031
- moved X20 124.0 mm to (165.1, 73.7), turned to 180 degrees
- moved X22 99.2 mm to (100.3, 104.1)
- moved X24 99.2 mm to (120.7, 104.1)
- moved X25 99.2 mm to (130.8, 104.1)
- moved X23 99.2 mm to (110.5, 104.1)
- moved X26 99.2 mm to (141.0, 104.1)
- moved X27 99.2 mm to (151.1, 104.1)
- moved X19 62.5 mm to (90.2, 73.7)
- moved C10 55.7 mm to (34.3, 78.7)
- moved OK1 55.7 mm to (34.3, 88.9)
- moved OK2 55.7 mm to (24.1, 88.9)
- moved OK3 55.7 mm to (54.6, 88.9)
- moved OK4 55.7 mm to (44.5, 88.9)
- moved OK5 55.7 mm to (74.9, 88.9)
- moved OK6 55.7 mm to (64.8, 88.9)
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Connections:
- new net DSTMOUT0: R40.1, X19.3
- new net DSTMOUT1: R41.1, X19.2
- new net DSTMOUT2: R42.1, X19.1
- new net DSTMOUT3: R43.1, X20.3
- new net DSTMOUT4: R44.1, X20.2
- new net DSTMOUT5: R45.1, X20.1
- new net N$21: R40.2, T1.1
- new net N$22: D1.A, K1.2, T1.2, T1.4
- new net N$23: R41.2, T2.1
- new net N$24: R43.2, T4.1
- new net N$25: D2.A, K2.2, T2.2, T2.4
- new net N$26: R42.2, T3.1
- new net N$27: D3.A, K3.2, T3.2, T3.4
- new net N$28: R44.2, T5.1
- new net N$29: D4.A, K4.2, T4.2, T4.4
- new net N$30: R45.2, T6.1
- new net N$31: D5.A, K5.2, T5.2, T5.4
- new net N$32: D6.A, K6.2, T6.2, T6.4
- net 5V: no longer X28.1, X29.1, X30.1
- net DOUT0+: now also K1.P; no longer X19.1
- net DOUT0-: now also K1.S; no longer X19.2
- net DOUT1+: now also K2.P; no longer X19.3
- net DOUT1-: now also K2.S; no longer X19.4
- net DOUT2+: now also K3.P; no longer X20.1
- net DOUT2-: now also K3.S; no longer X20.2
- net DOUT3+: now also K4.P; no longer X20.3
- net DOUT3-: now also K4.S; no longer X20.4
- net DOUT4+: now also K5.P; no longer X21.1
- net DOUT4-: now also K5.S; no longer X21.2
- net DOUT5+: now also K6.P; no longer X21.3
- net DOUT5-: now also K6.S; no longer X21.4
- net GND: now also T1.3, T2.3, T3.3, T4.3, T5.3, T6.3; no longer X28.2, X29.2, X30.2
- net VDD: now also D1.C, D2.C, D3.C, D4.C, D5.C, D6.C, K1.1, K2.1, K3.1, K4.1, K5.1, K6.1
Routing:
- net VDD: track 80.5 -> 370.3 mm
- net N$23: track 0.00 -> 85.0 mm
- net N$24: track 0.00 -> 71.0 mm
- net N$30: track 0.00 -> 66.9 mm
- net DOUT5+: track 13.2 -> 64.5 mm
- net DOUT3+: track 16.4 -> 63.0 mm
- net N$26: track 0.00 -> 45.0 mm
- net DOUT5-: track 13.2 -> 58.1 mm
- net DOUT3-: track 15.4 -> 59.2 mm
- net DOUT1+: track 21.8 -> 63.0 mm
- net DOUT1-: track 19.3 -> 60.2 mm
- net N$28: track 0.00 -> 37.1 mm
- net 5V: track 59.4 -> 26.0 mm
- net N$27: track 0.00 -> 19.6 mm
- net N$31: track 0.00 -> 19.4 mm
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Other:
- board text removed: "RELAY CONN"
- board text removed: "RELAY POWER"

Commit message: Few small changed and added gerbers
Parts:
- added D10, D7, D8, D9: BAS40, diode:SOT23
- added D11: 1N4004, diode:DO41-10
- added F1: FUSESHK20Q, fuse:SHK20Q
- moved J1 18.0 mm to (10.2, 71.1)
Connections:
- new net N$12: F1.1A, J1.3
- net AIN0: now also D7.3
- net AIN1: now also D9.3
- net AIN2: now also D8.3
- net AIN3: now also D10.3
- net GND: now also D10.1, D11.A, D7.1, D8.1, D9.1
- net VDD: now also D11.C, F1.2A; no longer J1.3
Routing:
- net N$12: track 0.00 -> 18.6 mm
- net VDD: track 370.3 -> 357.6 mm
- net AIN2: track 32.4 -> 38.4 mm
- net AIN1: track 23.7 -> 27.8 mm
- net AIN0: track 30.6 -> 34.6 mm
- net AIN3: track 37.1 -> 39.9 mm
Other:
- board text added: "3"
- board text added: "PRACA DYPLOMOWA MAGISTERSKA"
- board text added: "RELAY IN"
- board text added: "RELAY OUT"
- board text added: "REPOS: github.com\WojSkwie"
- board text added: "WOJCIECH SKWIERAWSKI"
