File: Magisterka/WeWyAn.sch (EAGLE design)
At the start: 65 parts, among them IC1 LM324N, IC2 LM1117T-3.3, IC4 LM324N, X10 22-23-2041, X11 22-23-2041, X4 22-23-2021

Commit message: Added board
Parts:
- added X18: (no value), con-molex:22-23-2061
- added X19, X20, X21, X22, X23, X24: 22-23-2031, con-molex:22-23-2031
Connections:
- net DSTMIN0: now also X18-6.S
- net DSTMIN1: now also X18-5.S
- net DSTMIN2: now also X18-4.S
- net DSTMIN3: now also X18-3.S
- net DSTMIN4: now also X18-2.S
- net DSTMIN5: now also X18-1.S
Changed lines of the file:
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@@
 <part name="X16" library="con-ptr500" deviceset="AK500/2-H" device=""/>
 <part name="X17" library="con-ptr500" deviceset="AK500/2-H" device=""/>
+<part name="X18" library="con-molex" library_urn="urn:adsk.eagle:library:165" deviceset="22-23-2061" device=""/>
+<part name="X19" library="con-molex" library_urn="urn:adsk.eagle:library:165" deviceset="22-23-2031" device=""/>
+<part name="X20" library="con-molex" library_urn="urn:adsk.eagle:library:165" deviceset="22-23-2031" device=""/>
+<part name="X21" library="con-molex" library_urn="urn:adsk.eagle:library:165" deviceset="22-23-2031" device=""/>
+<part name="X22" library="con-molex" library_urn="urn:adsk.eagle:library:165" deviceset="22-23-2031" device=""/>
+<part name="X23" library="con-molex" library_urn="urn:adsk.eagle:library:165" deviceset="22-23-2031" device=""/>
+<part name="X24" library="con-molex" library_urn="urn:adsk.eagle:library:165" deviceset="22-23-2031" device=""/>
 </parts>
 <sheets>
@@
 <wire x1="368.3" y1="-96.52" x2="205.74" y2="-96.52" width="0.1524" layer="97" style="longdash"/>
 <wire x1="205.74" y1="-96.52" x2="205.74" y2="2.54" width="0.1524" layer="97" style="longdash"/>
-<wire x1="-78.74" y1="-124.46" x2="157.48" y2="-124.46" width="0.1524" layer="97" style="longdash"/>
-<wire x1="160.02" y1="-124.46" x2="160.02" y2="-271.78" width="0.1524" layer="97" style="longdash"/>
+<wire x1="-78.74" y1="-124.46" x2="185.42" y2="-124.46" width="0.1524" layer="97" style="longdash"/>
+<wire x1="185.42" y1="-124.46" x2="185.42" y2="-271.78" width="0.1524" layer="97" style="longdash"/>
 <wire x1="-78.74" y1="-124.46" x2="-78.74" y2="-271.78" width="0.1524" layer="97" style="longdash"/>
-<wire x1="-78.74" y1="-271.78" x2="160.02" y2="-271.78" width="0.1524" layer="97" style="longdash"/>
+<wire x1="-78.74" y1="-271.78" x2="185.42" y2="-271.78" width="0.1524" layer="97" style="longdash"/>
 </plain>
 <instances>
@@
 <instance part="X17" gate="-1" x="-40.64" y="-223.52"/>
 <instance part="X17" gate="-2" x="-40.64" y="-228.6"/>
+<instance part="X18" gate="-1" x="160.02" y="-203.2" rot="R180"/>
+<instance part="X18" gate="-2" x="160.02" y="-200.66" rot="R180"/>
+<instance part="X18" gate="-3" x="160.02" y="-198.12" rot="R180"/>
+<instance part="X18" gate="-4" x="160.02" y="-195.58" rot="R180"/>
+<instance part="X18" gate="-5" x="160.02" y="-193.04" rot="R180"/>
+<instance part="X18" gate="-6" x="160.02" y="-190.5" rot="R180"/>
+<instance part="X19" gate="-1" x="220.98" y="-132.08"/>
+<instance part="X19" gate="-2" x="220.98" y="-134.62"/>
+<instance part="X19" gate="-3" x="220.98" y="-137.16"/>
+<instance part="X20" gate="-1" x="220.417490625" y="-146.101828125"/>
+<instance part="X20" gate="-2" x="220.417490625" y="-148.641828125"/>
+<instance part="X20" gate="-3" x="220.417490625" y="-151.181828125"/>
+<instance part="X21" gate="-1" x="223.52" y="-195.58"/>
+<instance part="X21" gate="-2" x="223.52" y="-198.12"/>
+<instance part="X21" gate="-3" x="223.52" y="-200.66"/>
+<instance part="X22" gate="-1" x="220.98" y="-220.98"/>
+<instance part="X22" gate="-2" x="220.98" y="-223.52"/>
+<instance part="X22" gate="-3" x="220.98" y="-226.06"/>
+<instance part="X23" gate="-1" x="220.98" y="-259.08"/>
+<instance part="X23" gate="-2" x="220.98" y="-261.62"/>
+<instance part="X23" gate="-3" x="220.98" y="-264.16"/>
+<instance part="X24" gate="-1" x="220.98" y="-292.1"/>
+<instance part="X24" gate="-2" x="220.98" y="-294.64"/>
+<instance part="X24" gate="-3" x="220.98" y="-297.18"/>
 </instances>
 <busses>
@@
 <label x="55.88" y="-195.58" size="1.016" layer="95" xref="yes"/>
 </segment>
+<segment>
+<pinref part="X18" gate="-4" pin="S"/>
+<wire x1="165.1" y1="-195.58" x2="162.56" y2="-195.58" width="0.1524" layer="91"/>
+<label x="165.1" y="-195.58" size="1.016" layer="95" xref="yes"/>
+</segment>
 </net>
 <net name="DIN4+" class="0">
@@
 <label x="55.88" y="-238.76" size="1.016" layer="95" xref="yes"/>
 </segment>
+<segment>
+<pinref part="X18" gate="-2" pin="S"/>
+<wire x1="165.1" y1="-200.66" x2="162.56" y2="-200.66" width="0.1524" layer="91"/>
+<label x="165.1" y="-200.66" size="1.016" layer="95" xref="yes"/>
+<label x="165.1" y="-200.66" size="1.016" layer="95" xref="yes"/>
+</segment>
 </net>
 <net name="DIN0-" class="0">
@@
 <label x="55.88" y="-149.86" size="1.016" layer="95" xref="yes"/>
 </segment>
+<segment>
+<pinref part="X18" gate="-6" pin="S"/>
+<wire x1="165.1" y1="-190.5" x2="162.56" y2="-190.5" width="0.1524" layer="91"/>
+<label x="165.1" y="-190.5" size="1.016" layer="95" xref="yes"/>
+</segment>
 </net>
 <net name="DIN1-" class="0">
@@
 <label x="134.62" y="-149.86" size="1.016" layer="95" xref="yes"/>
 </segment>
+<segment>
+<pinref part="X18" gate="-5" pin="S"/>
+<wire x1="165.1" y1="-193.04" x2="162.56" y2="-193.04" width="0.1524" layer="91"/>
+<label x="165.1" y="-193.04" size="1.016" layer="95" xref="yes"/>
+</segment>
 </net>
 <net name="DSTMIN3" class="0">
@@
 <label x="134.62" y="-195.58" size="1.016" layer="95" xref="yes"/>
 </segment>
+<segment>
+<pinref part="X18" gate="-3" pin="S"/>
+<wire x1="165.1" y1="-198.12" x2="162.56" y2="-198.12" width="0.1524" layer="91"/>
+<label x="165.1" y="-198.12" size="1.016" layer="95" xref="yes"/>
+</segment>
 </net>
 <net name="DIN3+" class="0">
@@
 <label x="134.62" y="-238.76" size="1.016" layer="95" xref="yes"/>
 </segment>
-</net>
+<segment>
+<pinref part="X18" gate="-1" pin="S"/>
+<wire x1="165.1" y1="-203.2" x2="162.56" y2="-203.2" width="0.1524" layer="91"/>
+<label x="165.1" y="-203.2" size="1.016" layer="95" xref="yes"/>
+</segment>
+</net>

Commit message: Most of digital part in schematics
Parts:
- removed IC2: LM1117T-3.3, lm1117:LM1117T-3.3
- added C1: 330n, rcl:C-EUC0603
- added C10, C11, C12, C13, C14, C8, C9: 100n, rcl:C-EUC0603
- added IC3: 7805TV, linear:7805TV
- added IC5: LM1117T-3.3-V, lm1117:LM1117T-3.3-V
- added X25, X26, X27: (no value), con-ptr500:AK500/2-H
- added X28, X29, X30: 22-23-2021, con-molex:22-23-2021
- X19, X20, X21: value 22-23-2031 -> 22-23-2041; device con-molex:22-23-2031 -> con-molex:22-23-2041
- X22, X23, X24: value 22-23-2031 -> (none); device con-molex:22-23-2031 -> con-ptr500:AK500/2-H
Connections:
- new net 5V: C3.1, C8.1, IC3.VO, IC5.IN, X28-1.S, X29-1.S, X30-1.S
- new net DOUT0+: X19-1.S, X22-1.KL
- new net DOUT0-: X19-2.S, X22-2.KL
- new net DOUT1+: X19-3.S, X23-1.KL
- new net DOUT1-: X19-4.S, X23-2.KL
- new net DOUT2+: X20-1.S, X24-1.KL
- new net DOUT2-: X20-2.S, X24-2.KL
- new net DOUT3+: X20-3.S, X25-1.KL
- new net DOUT3-: X20-4.S, X25-2.KL
- new net DOUT4+: X21-1.S, X26-1.KL
- new net DOUT4-: X21-2.S, X26-2.KL
- new net DOUT5+: X21-3.S, X27-1.KL
- new net DOUT5-: X21-4.S, X27-2.KL
- net DSTMIN0: now also C9.1
- net DSTMIN1: now also C10.1
- net DSTMIN2: now also C12.1
- net DSTMIN3: now also C11.1
- net DSTMIN4: now also C13.1
- net DSTMIN5: now also C14.1
- net GND: now also C1.2, C10.2, C11.2, C12.2, C13.2, C14.2, C8.2, C9.2, IC3.GND, IC5.GND, X28-2.S, X29-2.S, X30-2.S; no longer IC2.GND
- net VCC: now also IC5.OUT; no longer IC2.OUT
- net VDD: now also C1.1, IC3.VI; no longer C3.1, IC2.IN
Other:
- moved on the sheet: J1, X19-1, X19-2, X19-3, X20-1, X20-2, X20-3, X21-1, X21-2, X21-3, X22-1, X22-2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

Commit message: Pinswap in PWM CRIMP and moved several components
Parts:
- added X31: 22-23-2031, con-molex:22-23-2031
- R13, R14, R17, R20: value (none) -> 10k
- R16, R19, R22, R4: value (none) -> 20k
- X18: value (none) -> 22-23-2031; device con-molex:22-23-2061 -> con-molex:22-23-2031
Connections:
- net DSTMIN0: now also X18-3.S; no longer X18-6.S
- net DSTMIN1: now also X18-2.S; no longer X18-5.S
- net DSTMIN2: now also X18-1.S; no longer X18-4.S
- net DSTMIN3: now also X31-3.S; no longer X18-3.S
- net DSTMIN4: now also X31-2.S; no longer X18-2.S
- net DSTMIN5: now also X31-1.S; no longer X18-1.S
- net PWM0: now also X11-1.S; no longer X11-2.S
- net PWM1: now also X11-2.S; no longer X11-1.S
- net PWM2: now also X11-3.S; no longer X11-4.S
- net PWM3: now also X11-4.S; no longer X11-3.S
Other:
- moved on the sheet: X18-1, X18-2, X18-3
Changed lines of the file:
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@@
 <part name="GND8" library="supply1" deviceset="GND" device=""/>
 <part name="GND9" library="supply1" deviceset="GND" device=""/>
-<part name="R4" library="rcl" deviceset="R-EU_" device="R0603"/>
-<part name="R13" library="rcl" deviceset="R-EU_" device="R0603"/>
-<part name="R14" library="rcl" deviceset="R-EU_" device="R0603"/>
+<part name="R4" library="rcl" deviceset="R-EU_" device="R0603" value="20k"/>
+<part name="R13" library="rcl" deviceset="R-EU_" device="R0603" value="10k"/>
+<part name="R14" library="rcl" deviceset="R-EU_" device="R0603" value="10k"/>
 <part name="C4" library="rcl" deviceset="C-EU" device="C0603K" value="100n"/>
 <part name="C5" library="rcl" deviceset="C-EU" device="C0603K" value="100n"/>
@@
 <part name="C7" library="rcl" deviceset="C-EU" device="C0603K" value="100n"/>
 <part name="R15" library="rcl" deviceset="R-EU_" device="R0603" value="47k"/>
-<part name="R16" library="rcl" deviceset="R-EU_" device="R0603"/>
-<part name="R17" library="rcl" deviceset="R-EU_" device="R0603"/>
+<part name="R16" library="rcl" deviceset="R-EU_" device="R0603" value="20k"/>
+<part name="R17" library="rcl" deviceset="R-EU_" device="R0603" value="10k"/>
 <part name="R18" library="rcl" deviceset="R-EU_" device="R0603" value="47k"/>
-<part name="R19" library="rcl" deviceset="R-EU_" device="R0603"/>
-<part name="R20" library="rcl" deviceset="R-EU_" device="R0603"/>
+<part name="R19" library="rcl" deviceset="R-EU_" device="R0603" value="20k"/>
+<part name="R20" library="rcl" deviceset="R-EU_" device="R0603" value="10k"/>
 <part name="R21" library="rcl" deviceset="R-EU_" device="R0603" value="47k"/>
 <part name="GND10" library="supply1" deviceset="GND" device=""/>
@@
 <part name="GND16" library="supply1" deviceset="GND" device=""/>
 <part name="GND17" library="supply1" deviceset="GND" device=""/>
-<part name="R22" library="rcl" deviceset="R-EU_" device="R0603"/>
+<part name="R22" library="rcl" deviceset="R-EU_" device="R0603" value="20k"/>
 <part name="R23" library="rcl" deviceset="R-EU_" device="R0603" value="47k"/>
 <part name="X2" library="con-ptr500" deviceset="AK500/2-H" device=""/>
@@
 <part name="X16" library="con-ptr500" deviceset="AK500/2-H" device=""/>
 <part name="X17" library="con-ptr500" deviceset="AK500/2-H" device=""/>
-<part name="X18" library="con-molex" library_urn="urn:adsk.eagle:library:165" deviceset="22-23-2061" device=""/>
 <part name="X19" library="con-molex" library_urn="urn:adsk.eagle:library:165" deviceset="22-23-2041" device=""/>
 <part name="X20" library="con-molex" library_urn="urn:adsk.eagle:library:165" deviceset="22-23-2041" device=""/>
@@
 <part name="GND41" library="supply1" deviceset="GND" device=""/>
 <part name="IC5" library="lm1117" deviceset="LM1117T-*" device="-V" technology="3.3"/>
+<part name="X18" library="con-molex" library_urn="urn:adsk.eagle:library:165" deviceset="22-23-2031" device=""/>
+<part name="X31" library="con-molex" library_urn="urn:adsk.eagle:library:165" deviceset="22-23-2031" device=""/>
 </parts>
 <sheets>
@@
 <instance part="X17" gate="-1" x="-40.64" y="-223.52"/>
 <instance part="X17" gate="-2" x="-40.64" y="-228.6"/>
-<instance part="X18" gate="-1" x="160.02" y="-203.2" rot="R180"/>
-<instance part="X18" gate="-2" x="160.02" y="-200.66" rot="R180"/>
-<instance part="X18" gate="-3" x="160.02" y="-198.12" rot="R180"/>
-<instance part="X18" gate="-4" x="160.02" y="-195.58" rot="R180"/>
-<instance part="X18" gate="-5" x="160.02" y="-193.04" rot="R180"/>
-<instance part="X18" gate="-6" x="160.02" y="-190.5" rot="R180"/>
 <instance part="X19" gate="-1" x="238.76" y="-170.18"/>
 <instance part="X19" gate="-2" x="238.76" y="-172.72"/>
@@
 <instance part="GND41" gate="1" x="233.68" y="-162.56"/>
 <instance part="IC5" gate="G$1" x="-63.5" y="-7.62"/>
+<instance part="X18" gate="-1" x="160.02" y="-193.04" rot="R180"/>
+<instance part="X18" gate="-2" x="160.02" y="-190.5" rot="R180"/>
+<instance part="X18" gate="-3" x="160.02" y="-187.96" rot="R180"/>
+<instance part="X31" gate="-1" x="160.02" y="-203.2" rot="R180"/>
+<instance part="X31" gate="-2" x="160.02" y="-200.66" rot="R180"/>
+<instance part="X31" gate="-3" x="160.02" y="-198.12" rot="R180"/>
 </instances>
 <busses>
@@
 </segment>
 <segment>
-<pinref part="X11" gate="-2" pin="S"/>
-<wire x1="355.6" y1="-17.78" x2="353.06" y2="-17.78" width="0.1524" layer="91"/>
-<label x="355.6" y="-17.78" size="1.016" layer="95" xref="yes"/>
+<pinref part="X11" gate="-1" pin="S"/>
+<wire x1="355.6" y1="-20.32" x2="353.06" y2="-20.32" width="0.1524" layer="91"/>
+<label x="355.6" y="-20.32" size="1.016" layer="95" xref="yes"/>
 </segment>
 </net>
@@
 </segment>
 <segment>
+<pinref part="X11" gate="-3" pin="S"/>
+<wire x1="355.6" y1="-15.24" x2="353.06" y2="-15.24" width="0.1524" layer="91"/>
+<label x="355.6" y="-15.24" size="1.016" layer="95" xref="yes"/>
+</segment>
+</net>
+<net name="PWM3" class="0">
+<segment>
+<pinref part="R21" gate="G$1" pin="1"/>
+<wire x1="279.4" y1="-68.58" x2="281.94" y2="-68.58" width="0.1524" layer="91" style="longdash"/>
+<label x="279.4" y="-68.58" size="1.27" layer="95" rot="R180" xref="yes"/>
+</segment>
+<segment>
 <pinref part="X11" gate="-4" pin="S"/>
 <wire x1="355.6" y1="-12.7" x2="353.06" y2="-12.7" width="0.1524" layer="91"/>
 <label x="355.6" y="-12.7" size="1.016" layer="95" xref="yes"/>
-</segment>
-</net>
-<net name="PWM3" class="0">
-<segment>
-<pinref part="R21" gate="G$1" pin="1"/>
-<wire x1="279.4" y1="-68.58" x2="281.94" y2="-68.58" width="0.1524" layer="91" style="longdash"/>
-<label x="279.4" y="-68.58" size="1.27" layer="95" rot="R180" xref="yes"/>
-</segment>
-<segment>
-<pinref part="X11" gate="-3" pin="S"/>
-<wire x1="355.6" y1="-15.24" x2="353.06" y2="-15.24" width="0.1524" layer="91"/>
-<label x="355.6" y="-15.24" size="1.016" layer="95" xref="yes"/>
 </segment>
 </net>
@@
 </segment>
 <segment>
-<pinref part="X11" gate="-1" pin="S"/>
-<wire x1="355.6" y1="-20.32" x2="353.06" y2="-20.32" width="0.1524" layer="91"/>
-<label x="355.6" y="-20.32" size="1.016" layer="95" xref="yes"/>
+<pinref part="X11" gate="-2" pin="S"/>
+<wire x1="355.6" y1="-17.78" x2="353.06" y2="-17.78" width="0.1524" layer="91"/>
+<label x="355.6" y="-17.78" size="1.016" layer="95" xref="yes"/>
 </segment>
 </net>
@@
 </segment>
 <segment>
-<pinref part="X18" gate="-4" pin="S"/>
-<wire x1="165.1" y1="-195.58" x2="162.56" y2="-195.58" width="0.1524" layer="91"/>
-<label x="165.1" y="-195.58" size="1.016" layer="95" xref="yes"/>
+<wire x1="165.1" y1="-193.04" x2="162.56" y2="-193.04" width="0.1524" layer="91"/>
+<label x="165.1" y="-193.04" size="1.016" layer="95" xref="yes"/>
+<pinref part="X18" gate="-1" pin="S"/>
 </segment>
 </net>
@@
 </segment>
 <segment>
-<pinref part="X18" gate="-2" pin="S"/>
 <wire x1="165.1" y1="-200.66" x2="162.56" y2="-200.66" width="0.1524" layer="91"/>
 <label x="165.1" y="-200.66" size="1.016" layer="95" xref="yes"/>
 <label x="165.1" y="-200.66" size="1.016" layer="95" xref="yes"/>
+<pinref part="X31" gate="-2" pin="S"/>
 </segment>
 </net>
@@
 </segment>
 <segment>
-<pinref part="X18" gate="-6" pin="S"/>
-<wire x1="165.1" y1="-190.5" x2="162.56" y2="-190.5" width="0.1524" layer="91"/>
-<label x="165.1" y="-190.5" size="1.016" layer="95" xref="yes"/>
+<wire x1="165.1" y1="-187.96" x2="162.56" y2="-187.96" width="0.1524" layer="91"/>
+<label x="165.1" y="-187.96" size="1.016" layer="95" xref="yes"/>
+<pinref part="X18" gate="-3" pin="S"/>
 </segment>
 </net>
@@
 </segment>
 <segment>
-<pinref part="X18" gate="-5" pin="S"/>
-<wire x1="165.1" y1="-193.04" x2="162.56" y2="-193.04" width="0.1524" layer="91"/>
-<label x="165.1" y="-193.04" size="1.016" layer="95" xref="yes"/>
+<wire x1="165.1" y1="-190.5" x2="162.56" y2="-190.5" width="0.1524" layer="91"/>
+<label x="165.1" y="-190.5" size="1.016" layer="95" xref="yes"/>
+<pinref part="X18" gate="-2" pin="S"/>
 </segment>
 </net>
@@
 </segment>
 <segment>
-<pinref part="X18" gate="-3" pin="S"/>
 <wire x1="165.1" y1="-198.12" x2="162.56" y2="-198.12" width="0.1524" layer="91"/>
 <label x="165.1" y="-198.12" size="1.016" layer="95" xref="yes"/>
+<pinref part="X31" gate="-3" pin="S"/>
 </segment>
 </net>
@@
 </segment>
 <segment>
-<pinref part="X18" gate="-1" pin="S"/>
 <wire x1="165.1" y1="-203.2" x2="162.56" y2="-203.2" width="0.1524" layer="91"/>
 <label x="165.1" y="-203.2" size="1.016" layer="95" xref="yes"/>
-</segment>
-</net>
+<pinref part="X31" gate="-1" pin="S"/>
+</segment>
+</net>

Commit message: first final
Connections:
- net DIN0+: now also R1.1; no longer OK2.AC1
- net DIN0-: now also OK2.AC1; no longer R1.1
- net DIN1+: now also R3.1; no longer OK1.AC1
- net DIN1-: now also OK1.AC1; no longer R3.1
- net DIN2+: now also R2.1; no longer OK4.AC1
- net DIN2-: now also OK4.AC1; no longer R2.1
- net DIN3+: now also R24.1; no longer OK3.AC1
- net DIN3-: now also OK3.AC1; no longer R24.1
- net DIN4+: now also R29.1; no longer OK6.AC1
- net DIN4-: now also OK6.AC1; no longer R29.1
- net DIN5+: now also R30.1; no longer OK5.AC1
- net DIN5-: now also OK5.AC1; no longer R30.1
- net DSTMIN0: now also OK2.C, R25.1; no longer R25.2
- net DSTMIN1: now also OK1.C
- net DSTMIN2: now also OK4.C, R27.1; no longer R27.2
- net DSTMIN3: now also OK3.C, R28.1; no longer R28.2
- net DSTMIN4: now also OK6.C, R31.1; no longer R31.2
- net DSTMIN5: now also OK5.C, R32.1; no longer R32.2
- net VCC: now also R25.2, R27.2, R28.2, R31.2, R32.2; no longer OK1.C, OK2.C, OK3.C, OK4.C, OK5.C, OK6.C, R25.1, R27.1, R28.1, R31.1, R32.1
Other:
- moved on the sheet: R25, R26, R27, R28, R31, R32

Commit message: size changes
Changed lines of the file:
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@@
 <wire x1="261.62" y1="-30.48" x2="264.16" y2="-30.48" width="0.1524" layer="91" style="longdash"/>
 <junction x="261.62" y="-30.48"/>
-<label x="264.16" y="-30.48" size="1.27" layer="95" xref="yes"/>
+<label x="264.16" y="-30.48" size="1.016" layer="95" xref="yes"/>
 </segment>
 <segment>
 <pinref part="X8" gate="-1" pin="KL"/>
 <wire x1="355.6" y1="-33.02" x2="353.06" y2="-33.02" width="0.1524" layer="91" style="longdash"/>
-<label x="355.6" y="-33.02" size="1.27" layer="95" xref="yes"/>
+<label x="355.6" y="-33.02" size="1.016" layer="95" xref="yes"/>
 </segment>
 </net>
@@
 <pinref part="R15" gate="G$1" pin="1"/>
 <wire x1="223.52" y1="-33.02" x2="226.06" y2="-33.02" width="0.1524" layer="91" style="longdash"/>
-<label x="223.52" y="-33.02" size="1.27" layer="95" rot="R180" xref="yes"/>
+<label x="223.52" y="-33.02" size="1.016" layer="95" rot="R180" xref="yes"/>
 </segment>
 <segment>
@@
 <wire x1="261.62" y1="-66.04" x2="264.16" y2="-66.04" width="0.1524" layer="91" style="longdash"/>
 <junction x="261.62" y="-66.04"/>
-<label x="264.16" y="-66.04" size="1.27" layer="95" xref="yes"/>
+<label x="264.16" y="-66.04" size="1.016" layer="95" xref="yes"/>
 </segment>
 <segment>
@@
 <wire x1="314.96" y1="-66.04" x2="317.5" y2="-66.04" width="0.1524" layer="91" style="longdash"/>
 <junction x="314.96" y="-66.04"/>
-<label x="317.5" y="-66.04" size="1.27" layer="95" xref="yes"/>
+<label x="317.5" y="-66.04" size="1.016" layer="95" xref="yes"/>
 </segment>
 <segment>
@@
 <pinref part="R18" gate="G$1" pin="1"/>
 <wire x1="226.06" y1="-68.58" x2="228.6" y2="-68.58" width="0.1524" layer="91" style="longdash"/>
-<label x="226.06" y="-68.58" size="1.27" layer="95" rot="R180" xref="yes"/>
+<label x="226.06" y="-68.58" size="1.016" layer="95" rot="R180" xref="yes"/>
 </segment>
 <segment>
@@
 <pinref part="R21" gate="G$1" pin="1"/>
 <wire x1="279.4" y1="-68.58" x2="281.94" y2="-68.58" width="0.1524" layer="91" style="longdash"/>
-<label x="279.4" y="-68.58" size="1.27" layer="95" rot="R180" xref="yes"/>
+<label x="279.4" y="-68.58" size="1.016" layer="95" rot="R180" xref="yes"/>
 </segment>
 <segment>
@@
 <pinref part="R23" gate="G$1" pin="1"/>
 <wire x1="279.4" y1="-33.02" x2="281.94" y2="-33.02" width="0.1524" layer="91" style="longdash"/>
-<label x="279.4" y="-33.02" size="1.27" layer="95" rot="R180" xref="yes"/>
+<label x="279.4" y="-33.02" size="1.016" layer="95" rot="R180" xref="yes"/>
 </segment>
 <segment>
@@
 <wire x1="314.96" y1="-30.48" x2="317.5" y2="-30.48" width="0.1524" layer="91" style="longdash"/>
 <junction x="314.96" y="-30.48"/>
-<label x="317.5" y="-30.48" size="1.27" layer="95" xref="yes"/>
+<label x="317.5" y="-30.48" size="1.016" layer="95" xref="yes"/>
 </segment>
 <segment>
 <pinref part="X9" gate="-1" pin="KL"/>
 <wire x1="355.6" y1="-45.72" x2="353.06" y2="-45.72" width="0.1524" layer="91" style="longdash"/>
-<label x="355.6" y="-45.72" size="1.27" layer="95" xref="yes"/>
+<label x="355.6" y="-45.72" size="1.016" layer="95" xref="yes"/>
 </segment>
 </net>

Commit message: Added relays
Parts:
- added K1, K2, K3, K4, K5, K6: E3206S, relay:E3206S
Changed lines of the file:
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@@
 <part name="X18" library="con-molex" library_urn="urn:adsk.eagle:library:165" deviceset="22-23-2031" device=""/>
 <part name="X31" library="con-molex" library_urn="urn:adsk.eagle:library:165" deviceset="22-23-2031" device=""/>
+<part name="K1" library="relay" library_urn="urn:adsk.eagle:library:339" deviceset="E3206S" device="" package3d_urn="urn:adsk.eagle:package:24311/1"/>
+<part name="K2" library="relay" library_urn="urn:adsk.eagle:library:339" deviceset="E3206S" device="" package3d_urn="urn:adsk.eagle:package:24311/1"/>
+<part name="K3" library="relay" library_urn="urn:adsk.eagle:library:339" deviceset="E3206S" device="" package3d_urn="urn:adsk.eagle:package:24311/1"/>
+<part name="K4" library="relay" library_urn="urn:adsk.eagle:library:339" deviceset="E3206S" device="" package3d_urn="urn:adsk.eagle:package:24311/1"/>
+<part name="K5" library="relay" library_urn="urn:adsk.eagle:library:339" deviceset="E3206S" device="" package3d_urn="urn:adsk.eagle:package:24311/1"/>
+<part name="K6" library="relay" library_urn="urn:adsk.eagle:library:339" deviceset="E3206S" device="" package3d_urn="urn:adsk.eagle:package:24311/1"/>
 </parts>
 <sheets>
@@
 <instance part="X31" gate="-2" x="160.02" y="-200.66" rot="R180"/>
 <instance part="X31" gate="-3" x="160.02" y="-198.12" rot="R180"/>
+<instance part="K1" gate="1" x="411.48" y="-111.76"/>
+<instance part="K1" gate="2" x="426.72" y="-111.76"/>
+<instance part="K2" gate="1" x="411.48" y="-127"/>
+<instance part="K2" gate="2" x="426.72" y="-127"/>
+<instance part="K3" gate="1" x="411.48" y="-144.78"/>
+<instance part="K3" gate="2" x="426.72" y="-144.78"/>
+<instance part="K4" gate="1" x="411.48" y="-160.02"/>
+<instance part="K4" gate="2" x="426.72" y="-160.02"/>
+<instance part="K5" gate="1" x="411.48" y="-177.8"/>
+<instance part="K5" gate="2" x="426.72" y="-177.8"/>
+<instance part="K6" gate="1" x="411.48" y="-195.58"/>
+<instance part="K6" gate="2" x="426.72" y="-195.58"/>
 </instances>
 <busses>
