File: Magisterka/WeWyAn.sch (EAGLE design)
At the start: 94 parts, among them IC1 LM324N, IC3 7805TV, IC4 LM324N, IC5 LM1117T-3.3-V, K1 E3206S, K2 E3206S, K3 E3206S, K4 E3206S, K5 E3206S, K6 E3206S, X10 22-23-2041, X11 22-23-2041, X18 22-23-2031, X19 22-23-2041, X20 22-23-2041, X21 22-23-2041, X28 22-23-2021, X29 22-23-2021, X30 22-23-2021, X31 22-23-2031, X4 22-23-2021

Commit message: second final
Parts:
- removed X21: 22-23-2041, con-molex:22-23-2041
- removed X28, X29, X30: 22-23-2021, con-molex:22-23-2021
- added D1, D2, D3, D4, D5, D6: (no value), diode:DIODE-DO214AC
- added H1, H2, H3, H4: MOUNT-HOLE3.0, holes:MOUNT-HOLE3.0
- added R40, R41, R42, R43, R44, R45: (no value), rcl:R-EU_R0603
- added T1, T2, T3, T4, T5, T6: (no value), zetex:NPNSOT223
- X19, X20: value 22-23-2041 -> 22-23-2031; device con-molex:22-23-2041 -> con-molex:22-23-2031
Connections:
- new net DSTMOUT0: R40.1, X19-3.S
- new net DSTMOUT1: R41.1, X19-2.S
- new net DSTMOUT2: R42.1, X19-1.S
- new net DSTMOUT3: R43.1, X20-3.S
- new net DSTMOUT4: R44.1, X20-2.S
- new net DSTMOUT5: R45.1, X20-1.S
- new net N$21: R40.2, T1.B
- new net N$22: D1.A, K11.2, T1.C
- new net N$23: R41.2, T2.B
- new net N$24: R43.2, T4.B
- new net N$25: D2.A, K21.2, T2.C
- new net N$26: R42.2, T3.B
- new net N$27: D3.A, K31.2, T3.C
- new net N$28: R44.2, T5.B
- new net N$29: D4.A, K41.2, T4.C
- new net N$30: R45.2, T6.B
- new net N$31: D5.A, K51.2, T5.C
- new net N$32: D6.A, K61.2, T6.C
- net 5V: no longer X28-1.S, X29-1.S, X30-1.S
- net DOUT0+: now also K12.P; no longer X19-1.S
- net DOUT0-: now also K12.S; no longer X19-2.S
- net DOUT1+: now also K22.P; no longer X19-3.S
- net DOUT1-: now also K22.S; no longer X19-4.S
- net DOUT2+: now also K32.P; no longer X20-1.S
- net DOUT2-: now also K32.S; no longer X20-2.S
- net DOUT3+: now also K42.P; no longer X20-3.S
- net DOUT3-: now also K42.S; no longer X20-4.S
- net DOUT4+: now also K52.P; no longer X21-1.S
- net DOUT4-: now also K52.S; no longer X21-2.S
- net DOUT5+: now also K62.P; no longer X21-3.S
- net DOUT5-: now also K62.S; no longer X21-4.S
- net GND: now also T1.E, T2.E, T3.E, T4.E, T5.E, T6.E; no longer X28-2.S, X29-2.S, X30-2.S
- net VDD: now also D1.C, D2.C, D3.C, D4.C, D5.C, D6.C, K11.1, K21.1, K31.1, K41.1, K51.1, K61.1
Other:
- moved on the sheet: K1, K2, K3, K4, K5, K6, X19-1, X19-2, X19-3, X20-1, X20-2, X20-3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

Commit message: Few small changed and added gerbers
Parts:
- added D10, D7, D8, D9: BAS40, diode:BAS40
- added D11: 1N4004, diode:1N4004
- added F1: FUSESHK20Q, fuse:FUSESHK20Q
Connections:
- new net N$12: F1.1, J1.3
- net AIN0: now also D7.C
- net AIN1: now also D9.C
- net AIN2: now also D8.C
- net AIN3: now also D10.C
- net GND: now also D10.A, D11.A, D7.A, D8.A, D9.A
- net VDD: now also D11.C, F1.2; no longer J1.3
Other:
- moved on the sheet: IC4B, IC4D, R11, R12, R7, R8
